Commit message: All links placed

File: fanuc_description/robot/FANUC_M-20iA.urdf (robot description, URDF)
Before this commit: robot M-20iA, 6 links, 5 joints
Links:
- added link flange
- added link link5; collision mesh filename=package://${COLLISION_DIR}/link_5.stl; visual mesh filename=package://${VISUAL_DIR}/link_5.dae
- added link link6; collision mesh filename=package://${COLLISION_DIR}/link_6.stl; visual mesh filename=package://${VISUAL_DIR}/link_6.dae
Joints:
- added joint flange: type fixed, parent link6, child flange, origin xyz=0 0 0.1 rpy=0 0 0
- added joint joint5: type revolute, parent link4, child link5, origin xyz=0 0 0.51 rpy=${-pi/2} 0 0, axis 0 0 1, limit lower=-2.44 upper=2.44 effort=12 velocity=7.07
- added joint joint6: type revolute, parent link5, child link6, origin xyz=0 0 0 rpy=${pi/2} 0 0, axis 0 0 1, limit lower=-4.71 upper=4.71 effort=12 velocity=10.73
- joint joint4: limit lower=-3.49 upper=3.49 effort=12 velocity=6.28 -> lower=-3.49 upper=3.49 effort=12 velocity=7.07

Commit message: Now DH parameters are not hardcoded

File: fanuc_description/robot/FANUC_M-20iA.urdf (robot description, URDF)
Before this commit: robot M-20iA, 9 links, 8 joints
Joints:
- joint flange: origin xyz=0 0 0.1 rpy=0 0 0 -> xyz=0 0 ${dhparam['d'][5]} rpy=${dhparam['alpha'][5]} 0 ${dhparam['theta'][5]}
- joint joint2: origin xyz=0.15 0 0.525 rpy=${pi/2} 0 0 -> xyz=${-dhparam['a'][0]} 0 ${dhparam['d'][0]} rpy=${dhparam['alpha'][0]} 0 ${dhparam['theta'][0]}
- joint joint3: origin xyz=0 0.79 0 rpy=0 0 ${pi/2} -> xyz=0 ${dhparam['a'][1]} 0 rpy=${dhparam['alpha'][1]} 0 ${dhparam['theta'][1]}
- joint joint4: origin xyz=0.15 0 0 rpy=${pi/2} 0 0 -> xyz=${dhparam['a'][2]} 0 0 rpy=${dhparam['alpha'][2]} 0 ${dhparam['theta'][2]}
- joint joint5: origin xyz=0 0 0.51 rpy=${-pi/2} 0 0 -> xyz=0 0 0.51 rpy=${dhparam['alpha'][3]} 0 ${dhparam['theta'][3]}
- joint joint6: origin xyz=0 0 0 rpy=${pi/2} 0 0 -> xyz=0 0 0 rpy=${dhparam['alpha'][4]} 0 ${dhparam['theta'][4]}

Commit message: Offset corrections

File: fanuc_description/robot/FANUC_M-20iA.urdf (robot description, URDF)
Before this commit: robot M-20iA, 9 links, 8 joints
Joints:
- joint flange: origin xyz=0 0 ${dhparam['d'][5]} rpy=${dhparam['alpha'][5]} 0 ${dhparam['theta'][5]} -> xyz=${dhparam['a'][5]} 0 ${dhparam['d'][5]} rpy=${dhparam['alpha'][5]} 0 ${dhparam['theta'][5]}
- joint joint2: origin xyz=${-dhparam['a'][0]} 0 ${dhparam['d'][0]} rpy=${dhparam['alpha'][0]} 0 ${dhparam['theta'][0]} -> xyz=${dhparam['a'][0]} 0 ${dhparam['d'][0]} rpy=${dhparam['alpha'][0]} 0 ${dhparam['theta'][0]}
- joint joint3: origin xyz=0 ${dhparam['a'][1]} 0 rpy=${dhparam['alpha'][1]} 0 ${dhparam['theta'][1]} -> xyz=0 ${dhparam['a'][1]} ${dhparam['d'][1]} rpy=${dhparam['alpha'][1]} 0 ${dhparam['theta'][1]}
- joint joint4: limit lower=-3.49 upper=3.49 effort=12 velocity=7.07 -> lower=-3.49 upper=3.49 effort=20 velocity=7.07; origin xyz=${dhparam['a'][2]} 0 0 rpy=${dhparam['alpha'][2]} 0 ${dhparam['theta'][2]} -> xyz=${dhparam['a'][2]} 0 ${dhparam['d'][2]} rpy=${dhparam['alpha'][2]} 0 ${dhparam['theta'][2]}
- joint joint5: limit lower=-2.44 upper=2.44 effort=12 velocity=7.07 -> lower=-2.44 upper=2.44 effort=20 velocity=7.07; origin xyz=0 0 0.51 rpy=${dhparam['alpha'][3]} 0 ${dhparam['theta'][3]} -> xyz=0 ${dhparam['a'][3]} ${dhparam['d'][3]} rpy=${dhparam['alpha'][3]} 0 ${dhparam['theta'][3]}
- joint joint6: limit lower=-4.71 upper=4.71 effort=12 velocity=10.73 -> lower=-4.71 upper=4.71 effort=20 velocity=10.73; origin xyz=0 0 0 rpy=${dhparam['alpha'][4]} 0 ${dhparam['theta'][4]} -> xyz=${dhparam['a'][4]} 0 ${dhparam['d'][4]} rpy=${dhparam['alpha'][4]} 0 ${dhparam['theta'][4]}

Commit message: Now URDF file uses xacros

File: fanuc_description/robot/FANUC_M-20iA.urdf (robot description, URDF)
Before this commit: robot M-20iA, 9 links, 8 joints
Links:
- removed link base_link
- removed link flange
- removed link link1
- removed link link2
- removed link link3
- removed link link4
- removed link link5
- removed link link6
- removed link world
Joints:
- removed joint flange
- removed joint joint1
- removed joint joint2
- removed joint joint3
- removed joint joint4
- removed joint joint5
- removed joint joint6
- removed joint virtual_joint
