Commit message: package fanuc_moveit_config created

File: fanuc_description/robot/fanuc_m20ia.xacro (robot description, xacro)
@@ -5,5 +5,5 @@
 -->
 <!-- **************************************** FANUC M-20iA URDF **************************************** -->
-<robot name="M-20iA" xmlns:xacro="http://www.ros.org/wiki/xacro">
+<robot name="M20iA" xmlns:xacro="http://www.ros.org/wiki/xacro">
     <!-- **************************************** VARIABLES **************************************** -->
     <!-- This variable contains the DH parameters -->
@@ -47,5 +47,5 @@
     </xacro:macro>
     <!-- Macro for creating the flange -->
-    <xacro:macro name="create_flange" params="flange_name:='name' xyz:='0 0 0' rpy:='0 0 0' parent_link:='link6'" >
+    <xacro:macro name="create_flange" params="flange_name:='flange' xyz:='0 0 0' rpy:='0 0 0' parent_link:='link6'" >
         <link name="${flange_name}" />
         <joint name="${flange_name}" type="fixed">
@@ -98,5 +98,5 @@
     <!-- **************************************** LINKS **************************************** -->
     <!-- ******************** Used for fixing robot to Gazebo 'base_link' ******************** -->
-    <xacro:create_virtual_joint />
+    <!-- <xacro:create_virtual_joint /> -->
     <!-- ******************** BASE LINK  ******************** -->
     <xacro:link_joint index="0" />
